Commit message: gazebo setup

File: src/qp4_master/urdf/qp4.urdf (robot description, URDF)
Before this commit: robot qp4, 17 links, 16 joints
Links:
- removed link base_link
- added link torso_link, mass 1.0; collision mesh filename=file:///home/stewart/Robotics/ros-qp4/src/qp4_master/../../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 scale=0.001 0.001 0.001; collision mesh filename=file:///home/stewart/Robotics/ros-qp4/src/qp4_master/../../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 scale=0.001 0.001 0.001
- link back_left_femur_link: mass None -> 1.0; geometry collision mesh filename=file:///home/stewart/Robotics/ros-qp4/src/qp4_master/../../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 scale=0.001 0.001 0.001; collision mesh filename=file:///home/stewart/Robotics/ros-qp4/src/qp4_master/../../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 scale=0.001 0.001 0.001
- link back_left_foot_link: mass None -> 1.0; geometry collision mesh filename=file:///home/stewart/Robotics/ros-qp4/src/qp4_master/../../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 scale=0.001 0.001 0.001; visual mesh filename=file:///home/stewart/Robotics/ros-qp4/src/qp4_master/../../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 scale=0.001 0.001 0.001
- link back_left_hip_link: mass None -> 1.0; geometry collision mesh filename=file:///home/stewart/Robotics/ros-qp4/src/qp4_master/../../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 scale=0.001 0.001 0.001; collision mesh filename=file:///home/stewart/Robotics/ros-qp4/src/qp4_master/../../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 scale=0.001 0.001 0.001
- link back_left_tibia_link: mass None -> 1.0; geometry collision mesh filename=file:///home/stewart/Robotics/ros-qp4/src/qp4_master/../../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 scale=0.001 0.001 0.001; collision mesh filename=file:///home/stewart/Robotics/ros-qp4/src/qp4_master/../../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 scale=0.001 0.001 0.001
- link back_right_femur_link: mass None -> 1.0; geometry collision mesh filename=file:///home/stewart/Robotics/ros-qp4/src/qp4_master/../../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 scale=0.001 0.001 0.001; collision mesh filename=file:///home/stewart/Robotics/ros-qp4/src/qp4_master/../../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 scale=0.001 0.001 0.001
- link back_right_foot_link: mass None -> 1.0; geometry collision mesh filename=file:///home/stewart/Robotics/ros-qp4/src/qp4_master/../../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 scale=0.001 0.001 0.001; visual mesh filename=file:///home/stewart/Robotics/ros-qp4/src/qp4_master/../../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 scale=0.001 0.001 0.001
- link back_right_hip_link: mass None -> 1.0; geometry collision mesh filename=file:///home/stewart/Robotics/ros-qp4/src/qp4_master/../../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 scale=0.001 0.001 0.001; collision mesh filename=file:///home/stewart/Robotics/ros-qp4/src/qp4_master/../../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 scale=0.001 0.001 0.001
- link back_right_tibia_link: mass None -> 1.0; geometry collision mesh filename=file:///home/stewart/Robotics/ros-qp4/src/qp4_master/../../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 scale=0.001 0.001 0.001; collision mesh filename=file:///home/stewart/Robotics/ros-qp4/src/qp4_master/../../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 scale=0.001 0.001 0.001
- link front_left_femur_link: mass None -> 1.0; geometry collision mesh filename=file:///home/stewart/Robotics/ros-qp4/src/qp4_master/../../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 scale=0.001 0.001 0.001; collision mesh filename=file:///home/stewart/Robotics/ros-qp4/src/qp4_master/../../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 scale=0.001 0.001 0.001
- link front_left_foot_link: mass None -> 1.0; geometry collision mesh filename=file:///home/stewart/Robotics/ros-qp4/src/qp4_master/../../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 scale=0.001 0.001 0.001; visual mesh filename=file:///home/stewart/Robotics/ros-qp4/src/qp4_master/../../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 scale=0.001 0.001 0.001
- link front_left_hip_link: mass None -> 1.0; geometry collision mesh filename=file:///home/stewart/Robotics/ros-qp4/src/qp4_master/../../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 scale=0.001 0.001 0.001; collision mesh filename=file:///home/stewart/Robotics/ros-qp4/src/qp4_master/../../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 scale=0.001 0.001 0.001
- link front_left_tibia_link: mass None -> 1.0; geometry collision mesh filename=file:///home/stewart/Robotics/ros-qp4/src/qp4_master/../../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 scale=0.001 0.001 0.001; collision mesh filename=file:///home/stewart/Robotics/ros-qp4/src/qp4_master/../../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 scale=0.001 0.001 0.001
- link front_right_femur_link: mass None -> 1.0; geometry collision mesh filename=file:///home/stewart/Robotics/ros-qp4/src/qp4_master/../../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 scale=0.001 0.001 0.001; collision mesh filename=file:///home/stewart/Robotics/ros-qp4/src/qp4_master/../../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 scale=0.001 0.001 0.001
- link front_right_foot_link: mass None -> 1.0; geometry collision mesh filename=file:///home/stewart/Robotics/ros-qp4/src/qp4_master/../../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 scale=0.001 0.001 0.001; visual mesh filename=file:///home/stewart/Robotics/ros-qp4/src/qp4_master/../../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 scale=0.001 0.001 0.001
- link front_right_hip_link: mass None -> 1.0; geometry collision mesh filename=file:///home/stewart/Robotics/ros-qp4/src/qp4_master/../../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 scale=0.001 0.001 0.001; collision mesh filename=file:///home/stewart/Robotics/ros-qp4/src/qp4_master/../../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 scale=0.001 0.001 0.001
- link front_right_tibia_link: mass None -> 1.0; geometry collision mesh filename=file:///home/stewart/Robotics/ros-qp4/src/qp4_master/../../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 scale=0.001 0.001 0.001; collision mesh filename=file:///home/stewart/Robotics/ros-qp4/src/qp4_master/../../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 scale=0.001 0.001 0.001
Joints:
- removed joint back_left_femur_to_back_left_tibia
- removed joint back_left_hip_to_back_left_femur
- removed joint back_left_tibia_to_back_left_foot
- removed joint back_right_femur_to_back_right_tibia
- removed joint back_right_hip_to_back_right_femur
- removed joint back_right_tibia_to_back_right_foot
- removed joint base_to_back_left_hip
- removed joint base_to_back_right_hip
- removed joint base_to_front_left_hip
- removed joint base_to_front_right_hip
- removed joint front_left_femur_to_front_left_tibia
- removed joint front_left_hip_to_front_left_femur
- removed joint front_left_tibia_to_front_left_foot
- removed joint front_right_femur_to_front_right_tibia
- removed joint front_right_hip_to_front_right_femur
- removed joint front_right_tibia_to_front_right_foot
- added joint back_left_ankle_joint: type revolute, parent back_left_tibia_link, child back_left_foot_link, origin xyz=-0.0185 -0.0002 -0.077 rpy=0 0 0, limit lower=-3.14159265359 upper=3.14159265359 effort=10 velocity=1.0
- added joint back_left_hip_lateral_joint: type revolute, parent back_left_hip_link, child back_left_femur_link, origin xyz=-0.0192 0.0005 -0.0290 rpy=-1.57079632679 0 0, limit lower=-3.14159265359 upper=3.14159265359 effort=10 velocity=1.0
- added joint back_left_hip_swing_joint: type revolute, parent torso_link, child back_left_hip_link, origin xyz=-0.0398 0.0444 -0.0315, limit lower=-3.14159265359 upper=3.14159265359 effort=10 velocity=1.0
- added joint back_left_knee_joint: type revolute, parent back_left_femur_link, child back_left_tibia_link, origin xyz=0.019 0.0572 0 rpy=1.57079632679 0 0, limit lower=-3.14159265359 upper=3.14159265359 effort=10 velocity=1.0
- added joint back_right_ankle_joint: type revolute, parent back_right_tibia_link, child back_right_foot_link, origin xyz=0.0185 -0.0002 -0.077 rpy=0 0 0, limit lower=-3.14159265359 upper=3.14159265359 effort=10 velocity=1.0
- added joint back_right_hip_lateral_joint: type revolute, parent back_right_hip_link, child back_right_femur_link, origin xyz=0.0192 0.0005 -0.0290 rpy=-1.57079632679 0 0, limit lower=-3.14159265359 upper=3.14159265359 effort=10 velocity=1.0
- added joint back_right_hip_swing_joint: type revolute, parent torso_link, child back_right_hip_link, origin xyz=0.0398 0.0444 -0.0315, limit lower=-3.14159265359 upper=3.14159265359 effort=10 velocity=1.0
- added joint back_right_knee_joint: type revolute, parent back_right_femur_link, child back_right_tibia_link, origin xyz=-0.019 0.0572 0 rpy=1.57079632679 0 0, limit lower=-3.14159265359 upper=3.14159265359 effort=10 velocity=1.0
- added joint front_left_ankle_joint: type revolute, parent front_left_tibia_link, child front_left_foot_link, origin xyz=-0.0185 0.0002 -0.077 rpy=0 0 0, limit lower=-3.14159265359 upper=3.14159265359 effort=10 velocity=1.0
- added joint front_left_hip_lateral_joint: type revolute, parent front_left_hip_link, child front_left_femur_link, origin xyz=-0.0192 0.0005 -0.0290 rpy=-1.57079632679 0 0, limit lower=-3.14159265359 upper=3.14159265359 effort=10 velocity=1.0
- added joint front_left_hip_swing_joint: type revolute, parent torso_link, child front_left_hip_link, origin xyz=-0.0398 0.2984 -0.0315, limit lower=-3.14159265359 upper=3.14159265359 effort=10 velocity=1.0
- added joint front_left_knee_joint: type revolute, parent front_left_femur_link, child front_left_tibia_link, origin xyz=0.019 0.0572 0 rpy=1.57079632679 0 0, limit lower=-3.14159265359 upper=3.14159265359 effort=10 velocity=1.0
- added joint front_right_ankle_joint: type revolute, parent front_right_tibia_link, child front_right_foot_link, origin xyz=0.0185 0.0002 -0.077 rpy=0 0 0, limit lower=-3.14159265359 upper=3.14159265359 effort=10 velocity=1.0
- added joint front_right_hip_lateral_joint: type revolute, parent front_right_hip_link, child front_right_femur_link, origin xyz=0.0192 0.0005 -0.0290 rpy=-1.57079632679 0 0, limit lower=-3.14159265359 upper=3.14159265359 effort=10 velocity=1.0
- added joint front_right_hip_swing_joint: type revolute, parent torso_link, child front_right_hip_link, origin xyz=0.0398 0.2984 -0.0315, limit lower=-3.14159265359 upper=3.14159265359 effort=10 velocity=1.0
- added joint front_right_knee_joint: type revolute, parent front_right_femur_link, child front_right_tibia_link, origin xyz=-0.019 0.0572 0 rpy=1.57079632679 0 0, limit lower=-3.14159265359 upper=3.14159265359 effort=10 velocity=1.0

File: src/qp4_master/urdf/qp4.xacro (robot description, xacro)
@@ -12,4 +12,5 @@
     </xacro:macro>
     <xacro:include filename="$(find qp4_master)/urdf/qp4_materials.xacro"/>
+    <xacro:include filename="$(find qp4_master)/urdf/qp4_gazebo.xacro"/>
     <xacro:include filename="$(find qp4_master)/urdf/qp4_parts.xacro"/>
 </robot>

File: src/qp4_master/urdf/qp4_gazebo.xacro (robot description, xacro)
@@ -8,59 +8,11 @@
         </plugin>
     </gazebo>
-    <xacro:macro name="shoulder_swing_joint_gazebo" params="prefix">
-        <transmission name="${prefix}_shoulder_swing_joint_tran">
+    <xacro:macro name="hip_swing_joint_gazebo" params="prefix">
+        <transmission name="${prefix}_hip_swing_joint_tran">
             <type>transmission_interface/SimpleTransmission</type>
-            <joint name="${prefix}_shoulder_swing_joint">
+            <joint name="${prefix}_hip_swing_joint">
                 <hardwareInterface>EffortJointInterface</hardwareInterface>
             </joint>
-            <actuator name="${prefix}_shoulder_swing_joint_motor">
-                <hardwareInterface>EffortJointInterface</hardwareInterface>
-                <mechanicalReduction>1</mechanicalReduction>
-            </actuator>
-        </transmission>
-    </xacro:macro>
-    <xacro:macro name="shoulder_lateral_joint_gazebo" params="prefix">
-        <transmission name="${prefix}_shoulder_lateral_joint_tran">
-            <type>transmission_interface/SimpleTransmission</type>
-            <joint name="${prefix}_shoulder_lateral_joint">
-                <hardwareInterface>EffortJointInterface</hardwareInterface>
-            </joint>
-            <actuator name="${prefix}_shoulder_lateral_joint_motor">
-                <hardwareInterface>EffortJointInterface</hardwareInterface>
-                <mechanicalReduction>1</mechanicalReduction>
-            </actuator>
-        </transmission>
-    </xacro:macro>
-    <xacro:macro name="elbow_joint_gazebo" params="prefix">
-        <transmission name="${prefix}_elbow_joint_tran">
-            <type>transmission_interface/SimpleTransmission</type>
-            <joint name="${prefix}_elbow_joint">
-                <hardwareInterface>EffortJointInterface</hardwareInterface>
-            </joint>
-            <actuator name="${prefix}_elbow_joint_motor">
-                <hardwareInterface>EffortJointInterface</hardwareInterface>
-                <mechanicalReduction>1</mechanicalReduction>
-            </actuator>
-        </transmission>
-    </xacro:macro>
-    <xacro:macro name="hand_joint_gazebo" params="prefix">
-        <transmission name="${prefix}_elbow_joint_tran">
-            <type>transmission_interface/SimpleTransmission</type>
-            <joint name="${prefix}_elbow_joint">
-                <hardwareInterface>EffortJointInterface</hardwareInterface>
-            </joint>
-            <actuator name="${prefix}_elbow_joint_motor">
-                <hardwareInterface>EffortJointInterface</hardwareInterface>
-                <mechanicalReduction>1</mechanicalReduction>
-            </actuator>
-        </transmission>
-    </xacro:macro>
-    <xacro:macro name="hip_twist_joint_gazebo" params="prefix">
-        <transmission name="${prefix}_hip_twist_joint_tran">
-            <type>transmission_interface/SimpleTransmission</type>
-            <joint name="${prefix}_hip_twist_joint">
-                <hardwareInterface>EffortJointInterface</hardwareInterface>
-            </joint>
-            <actuator name="${prefix}_hip_twist_joint_motor">
+            <actuator name="${prefix}_hip_swing_joint_motor">
                 <hardwareInterface>EffortJointInterface</hardwareInterface>
                 <mechanicalReduction>1</mechanicalReduction>
@@ -80,16 +32,4 @@
         </transmission>
     </xacro:macro>
-    <xacro:macro name="hip_swing_joint_gazebo" params="prefix">
-        <transmission name="${prefix}_hip_swing_joint_tran">
-            <type>transmission_interface/SimpleTransmission</type>
-            <joint name="${prefix}_hip_swing_joint">
-                <hardwareInterface>EffortJointInterface</hardwareInterface>
-            </joint>
-            <actuator name="${prefix}_hip_swing_joint_motor">
-                <hardwareInterface>EffortJointInterface</hardwareInterface>
-                <mechanicalReduction>1</mechanicalReduction>
-            </actuator>
-        </transmission>
-    </xacro:macro>
     <xacro:macro name="knee_joint_gazebo" params="prefix">
         <transmission name="${prefix}_knee_joint_tran">
@@ -104,11 +44,11 @@
         </transmission>
     </xacro:macro>
-    <xacro:macro name="ankle_swing_joint_gazebo" params="prefix">
-        <transmission name="${prefix}_ankle_swing_joint_tran">
+    <xacro:macro name="ankle_joint_gazebo" params="prefix">
+        <transmission name="${prefix}_ankle_joint_tran">
             <type>transmission_interface/SimpleTransmission</type>
-            <joint name="${prefix}_ankle_swing_joint">
+            <joint name="${prefix}_ankle_joint">
                 <hardwareInterface>EffortJointInterface</hardwareInterface>
             </joint>
-            <actuator name="${prefix}_ankle_swing_joint_motor">
+            <actuator name="${prefix}_ankle_joint_motor">
                 <hardwareInterface>EffortJointInterface</hardwareInterface>
                 <mechanicalReduction>1</mechanicalReduction>
@@ -116,49 +56,19 @@
         </transmission>
     </xacro:macro>
-    <xacro:macro name="ankle_lateral_joint_gazebo" params="prefix">
-        <transmission name="${prefix}_ankle_lateral_joint_tran">
-            <type>transmission_interface/SimpleTransmission</type>
-            <joint name="${prefix}_ankle_lateral_joint">
-                <hardwareInterface>EffortJointInterface</hardwareInterface>
-            </joint>
-            <actuator name="${prefix}_ankle_lateral_joint_motor">
-                <hardwareInterface>EffortJointInterface</hardwareInterface>
-                <mechanicalReduction>1</mechanicalReduction>
-            </actuator>
-        </transmission>
-    </xacro:macro>
-    <xacro:macro name="foot_joint_gazebo" params="prefix">
-        <transmission name="${prefix}_ankle_lateral_joint_tran">
-            <type>transmission_interface/SimpleTransmission</type>
-            <joint name="${prefix}_ankle_lateral_joint">
-                <hardwareInterface>EffortJointInterface</hardwareInterface>
-            </joint>
-            <actuator name="${prefix}_ankle_lateral_joint_motor">
-                <hardwareInterface>EffortJointInterface</hardwareInterface>
-                <mechanicalReduction>1</mechanicalReduction>
-            </actuator>
-        </transmission>
-    </xacro:macro>
-    <shoulder_swing_joint_gazebo prefix="right"/>
-    <shoulder_swing_joint_gazebo prefix="left"/>
-    <shoulder_lateral_joint_gazebo prefix="right"/>
-    <shoulder_lateral_joint_gazebo prefix="left"/>
-    <elbow_joint_gazebo prefix="right"/>
-    <elbow_joint_gazebo prefix="left"/>
-    <hand_joint_gazebo prefix="right"/>
-    <hand_joint_gazebo prefix="left"/>
-    <hip_twist_joint_gazebo prefix="right"/>
-    <hip_twist_joint_gazebo prefix="left"/>
-    <hip_lateral_joint_gazebo prefix="right"/>
-    <hip_lateral_joint_gazebo prefix="left"/>
-    <hip_swing_joint_gazebo prefix="right"/>
-    <hip_swing_joint_gazebo prefix="left"/>
-    <knee_joint_gazebo prefix="right"/>
-    <knee_joint_gazebo prefix="left"/>
-    <ankle_swing_joint_gazebo prefix="right"/>
-    <ankle_swing_joint_gazebo prefix="left"/>
-    <ankle_lateral_joint_gazebo prefix="right"/>
-    <ankle_lateral_joint_gazebo prefix="left"/>
-    <foot_joint_gazebo prefix="right"/>
-    <foot_joint_gazebo prefix="left"/>
+    <hip_swing_joint_gazebo prefix="back_right"/>
+    <hip_swing_joint_gazebo prefix="back_left"/>
+    <hip_swing_joint_gazebo prefix="front_right"/>
+    <hip_swing_joint_gazebo prefix="front_left"/>
+    <hip_lateral_joint_gazebo prefix="back_right"/>
+    <hip_lateral_joint_gazebo prefix="back_left"/>
+    <hip_lateral_joint_gazebo prefix="front_right"/>
+    <hip_lateral_joint_gazebo prefix="front_left"/>
+    <knee_joint_gazebo prefix="back_right"/>
+    <knee_joint_gazebo prefix="back_left"/>
+    <knee_joint_gazebo prefix="front_right"/>
+    <knee_joint_gazebo prefix="front_left"/>
+    <ankle_joint_gazebo prefix="back_right"/>
+    <ankle_joint_gazebo prefix="back_left"/>
+    <ankle_joint_gazebo prefix="front_right"/>
+    <ankle_joint_gazebo prefix="front_left"/>
 </robot>
