Commit message: refactored for description package

File: src/qp4_description/urdf/qp4_parts.xacro (robot description, xacro)
@@ -16,42 +16,60 @@
 		<visual>
             <xacro:default_geometry cad_file="asb-512"/>
-            <origin rpy="${pi/2} 0 0"/>
+            <origin xyz="0 -0.1524 0" rpy="${pi/2} 0 0"/>
+		</visual>
+		<visual>
+            <xacro:default_geometry cad_file="asb-11"/>
+            <origin xyz="-0.0125 -0.127 -0.0127" rpy="0 0 ${pi/2}"/>
 		</visual>
         <visual>
             <xacro:default_geometry cad_file="asb-11"/>
-            <origin xyz="-0.0125 0.0254 -0.0127" rpy="0 0 ${pi/2}"/>
-	   </visual>
+            <origin xyz="0.0125 -0.127 -0.0127" rpy="0 0 -${pi/2}"/>
+		</visual>
         <visual>
             <xacro:default_geometry cad_file="asb-11"/>
-            <origin xyz="0.0125 0.0254 -0.0127" rpy="0 0 -${pi/2}"/>
-	   </visual>
+            <origin xyz="-0.0125 0.127 -0.0127" rpy="0 0 ${pi/2}"/>
+		</visual>
         <visual>
             <xacro:default_geometry cad_file="asb-11"/>
-            <origin xyz="-0.0125 0.2794 -0.0127" rpy="0 0 ${pi/2}"/>
-	   </visual>
-        <visual>
-            <xacro:default_geometry cad_file="asb-11"/>
-            <origin xyz="0.0125 0.2794 -0.0127" rpy="0 0 -${pi/2}"/>
-	   </visual>
-	 	<collision>
-            <xacro:default_geometry cad_file="asb-512"/>
-            <origin rpy="${pi/2} 0 0"/>
-		</collision>
-        <collision>
-            <xacro:default_geometry cad_file="asb-11"/>
-            <origin xyz="-0.0125 0.0254 -0.0127" rpy="0 0 ${pi/2}"/>
-	   </collision>
-        <collision>
-            <xacro:default_geometry cad_file="asb-11"/>
-            <origin xyz="0.0125 0.0254 -0.0127" rpy="0 0 -${pi/2}"/>
-	   </collision>
-        <collision>
-            <xacro:default_geometry cad_file="asb-11"/>
-            <origin xyz="-0.0125 0.2794 -0.0127" rpy="0 0 ${pi/2}"/>
-	   </collision>
-        <collision>
-            <xacro:default_geometry cad_file="asb-11"/>
-            <origin xyz="0.0125 0.2794 -0.0127" rpy="0 0 -${pi/2}"/>
-	   </collision>
+            <origin xyz="0.0125 0.127 -0.0127" rpy="0 0 -${pi/2}"/>
+		</visual>
+		<!--
+		   	<visual>
+	   			<geometry>
+					 <box size="0.1016 0.3048 0.0254"/>
+	   			</geometry>
+				<origin xyz="0 0 -0.0127"/>
+	   		</visual>
+		   	<visual>
+	   			<geometry>
+					 <box size="0.0508 0.3048 0.0254"/>
+	   			</geometry>
+				<origin xyz="-0.0508 0 -0.0254"/>
+	   		</visual>
+		   	<visual>
+	   			<geometry>
+					 <box size="0.0508 0.3048 0.0254"/>
+	   			</geometry>
+				<origin xyz="0.0508 0 -0.0254"/>
+	   		</visual>
+		-->
+	    <collision>
+   			<geometry>
+				 <box size="0.1016 0.3048 0.0254"/>
+   			</geometry>
+			<origin xyz="0 0 -0.0127"/>
+   		</collision>
+       	<collision>
+   			<geometry>
+				 <box size="0.0508 0.3048 0.0254"/>
+   			</geometry>
+			<origin xyz="-0.0508 0 -0.0254"/>
+   		</collision>
+       	<collision>
+   			<geometry>
+				 <box size="0.0508 0.3048 0.0254"/>
+   			</geometry>
+			<origin xyz="0.0508 0 -0.0254"/>
+   		</collision>
         <inertial>
           <origin xyz="0 0 0"/>
@@ -64,36 +82,24 @@
 		<!-- Hip -->
 		<link name="${prefix}_hip_link">
-	 		<visual>
-		        <xacro:default_geometry cad_file="hs-645-mg"/>
-		        <origin xyz="${reflectx*(0.01)} 0 0" rpy="0 ${reflectx*(-(pi/2))} ${reflectx*(pi/2)}"/>
-			</visual>
-			 <visual>
-		        <xacro:default_geometry cad_file="asb-04"/>
-		        <origin xyz="${reflectx*(0.01)} -0.0127 -0.0145" rpy="${pi/2} 0 ${reflectx*(pi)}"/>
-			</visual>
-			<visual>
-		        <xacro:default_geometry cad_file="asb-04"/>
-		        <origin xyz="${reflectx*(0.0129)} -0.0098 -0.0145" rpy="-${pi/2} 0 ${reflectx*(pi/2)}"/>
-			</visual>
-		    <visual>
-		        <xacro:default_geometry cad_file="hs-645-mg"/>
-		        <origin xyz="0 -0.0098 -0.029" rpy="${pi/2} ${reflectx*(pi/2)} ${reflectx*(pi/2)}"/>
-			</visual>
-	 		<collision>
-		        <xacro:default_geometry cad_file="hs-645-mg"/>
-		        <origin xyz="${reflectx*(0.01)} 0 0" rpy="0 ${reflectx*(-(pi/2))} ${reflectx*(pi/2)}"/>
-			</collision>
-			 <collision>
-		        <xacro:default_geometry cad_file="asb-04"/>
-		        <origin xyz="${reflectx*(0.01)} -0.0127 -0.0145" rpy="${pi/2} 0 ${reflectx*(pi)}"/>
-			</collision>
-			<collision>
-		        <xacro:default_geometry cad_file="asb-04"/>
-		        <origin xyz="${reflectx*(0.0129)} -0.0098 -0.0145" rpy="-${pi/2} 0 ${reflectx*(pi/2)}"/>
-			</collision>
-		    <collision>
-		        <xacro:default_geometry cad_file="hs-645-mg"/>
-		        <origin xyz="0 -0.0098 -0.029" rpy="${pi/2} ${reflectx*(pi/2)} ${reflectx*(pi/2)}"/>
-			</collision>
+			<visual>
+			 	<geometry>
+		       		<mesh filename="${cad_dir}/${prefix}_hip_s.dae" />
+			 	</geometry>
+			 	<origin xyz="${reflectx*(0.01)} ${0.01 + (reflecty*(-0.01))} 0" rpy="0 0 0"/>
+			</visual>
+			<!--
+			   	<visual>
+		   			<geometry>
+						 <box size="0.06 0.06 0.06"/>
+		   			</geometry>
+					<origin xyz="${reflectx*(0.01)} ${ (reflecty*(-0.01))} -0.0128"/>
+		   		</visual>
+			-->
+		   	<collision>
+	   			<geometry>
+					 <box size="0.06 0.06 0.06"/>
+	   			</geometry>
+				<origin xyz="${reflectx*(0.01)} ${ (reflecty*(-0.01))} -0.0128"/>
+	   		</collision>
 		    <inertial>
 		      <origin xyz="0 0 0"/>
@@ -105,5 +111,6 @@
 			<parent link="torso_link"/>
 			<child link="${prefix}_hip_link"/>
-			<origin xyz="${reflectx*(0.0398)} ${0.0444 + (0.254/2) + -reflecty*(0.254/2)} -0.0315" />
+			<origin xyz="${reflectx*(0.0395)} ${-reflecty*( (0.245/2) - 0.013)} -0.0315" rpy="0 0 0"/>
+			<axis xyz="0 ${-reflectx} 0" />
 			<limit lower="${-pi}" upper="${pi}" effort="10" velocity="1.0"/>
 	  	</joint>
@@ -118,12 +125,18 @@
 			    <origin xyz="0 0.0287 0" rpy="${reflectx*(pi)} 0 0"/>
 			</visual>
-			<collision>
-			    <xacro:default_geometry cad_file="asb-09-black"/>
-			    <origin xyz="0 0.0287 0" rpy="0 0 0"/>
-			</collision>
-			<collision>
-			    <xacro:default_geometry cad_file="asb-09-black"/>
-			    <origin xyz="0 0.0287 0" rpy="${reflectx*(pi)} 0 0"/>
-			</collision>
+			<!--
+			   	<visual>
+		   			<geometry>
+						 <box size="0.0525 0.085 0.0254"/>
+		   			</geometry>
+					<origin xyz="0 0.028 0"/>
+		   		</visual>
+			-->
+		   	<collision>
+	   			<geometry>
+					 <box size="0.0525 0.085 0.0254"/>
+	   			</geometry>
+				<origin xyz="0 0.028 0"/>
+	   		</collision>
 		    <inertial>
 		      <origin xyz="0 0 0"/>
@@ -152,16 +165,18 @@
 		        <origin xyz="0.0 0 -0.067" rpy="-${pi/2} 0 ${reflectx*(-(pi/2))}"/>
 			</visual>
-			<collision>
-			    <xacro:default_geometry cad_file="asb-15-black"/>
-			    <origin xyz="${reflectx*(-0.0043)} -0.01422 -0.0386" rpy="0 ${reflectx*(-(pi/2))} 0 "/>
-			</collision>
-		 	<collision>
-		        <xacro:default_geometry cad_file="hs-645-mg"/>
-		        <origin xyz="0.0 0 -0.01" rpy="${pi/2} 0 ${reflectx*(pi/2)}"/>
-			</collision>
-		 	<collision>
-		        <xacro:default_geometry cad_file="hs-645-mg"/>
-		        <origin xyz="0.0 0 -0.067" rpy="-${pi/2} 0 ${reflectx*(-(pi/2))}"/>
-			</collision>
+			<!--
+			   	<visual>
+		   			<geometry>
+						 <box size="0.0525 0.0254 0.115"/>
+		   			</geometry>
+					<origin xyz="${reflectx*(0.02)} 0 -0.039"/>
+		   		</visual>
+			-->
+		   	<collision>
+	   			<geometry>
+					 <box size="0.0525 0.0254 0.115"/>
+	   			</geometry>
+				<origin xyz="${reflectx*(0.02)} 0 -0.039"/>
+	   		</collision>
 		    <inertial>
 		      <origin xyz="0 0 0"/>
@@ -182,8 +197,18 @@
 				<origin xyz="0 0.0185 -0.0272" rpy="${pi/2} 0 ${pi}" />
 			</visual>
-			<collision>
-				<xacro:default_geometry cad_file="asb-11"/>
-				<origin xyz="0 0.0185 -0.0272" rpy="${pi/2} 0 ${pi}" />
-			</collision>
+			<!--
+			   	<visual>
+		   			<geometry>
+						 <box size="0.0523 0.0508 0.0400"/>
+		   			</geometry>
+					<origin xyz="0 0.01 -0.0072"/>
+		   		</visual>
+			-->
+		   	<collision>
+	   			<geometry>
+					 <box size="0.0523 0.0508 0.0400"/>
+	   			</geometry>
+				<origin xyz="0 0.01 -0.0072"/>
+	   		</collision>
 		    <inertial>
 		      <origin xyz="0 0 0"/>
