Commit message: refactoring

File: src/qp4_description/urdf/qp4.urdf (robot description, URDF)
Before this commit: robot qp4, 18 links, 17 joints
Links:
- link torso_link: geometry collision box size=0.028 0.3 0.0254; collision box size=0.08 0.06 0.0254

File: src/qp4_description/urdf/qp4_parts.xacro (robot description, xacro)
@@ -34,27 +34,7 @@
             <origin xyz="0.0125 0.127 -0.0127" rpy="0 0 -${pi/2}"/>
 		</visual>
-		<!--
-		   	<visual>
-	   			<geometry>
-					 <box size="0.1016 0.3048 0.0254"/>
-	   			</geometry>
-				<origin xyz="0 0 -0.0127"/>
-	   		</visual>
-		   	<visual>
-	   			<geometry>
-					 <box size="0.0508 0.3048 0.0254"/>
-	   			</geometry>
-				<origin xyz="-0.0508 0 -0.0254"/>
-	   		</visual>
-		   	<visual>
-	   			<geometry>
-					 <box size="0.0508 0.3048 0.0254"/>
-	   			</geometry>
-				<origin xyz="0.0508 0 -0.0254"/>
-	   		</visual>
-		-->
 	    <collision>
    			<geometry>
-				 <box size="0.1016 0.3048 0.0254"/>
+				 <box size="0.028 0.3 0.0254"/>
    			</geometry>
 			<origin xyz="0 0 -0.0127"/>
@@ -62,13 +42,13 @@
        	<collision>
    			<geometry>
-				 <box size="0.0508 0.3048 0.0254"/>
+				<box size="0.08 0.06 0.0254"/>
    			</geometry>
-			<origin xyz="-0.0508 0 -0.0254"/>
+			<origin xyz="0 -0.123 -0.0127"/>
    		</collision>
-       	<collision>
+		<collision>
    			<geometry>
-				 <box size="0.0508 0.3048 0.0254"/>
+				<box size="0.08 0.06 0.0254"/>
    			</geometry>
-			<origin xyz="0.0508 0 -0.0254"/>
+			<origin xyz="0 0.123 -0.0127"/>
    		</collision>
         <inertial>
@@ -88,12 +68,4 @@
 			 	<origin xyz="${reflectx*(0.01)} ${0.01 + (reflecty*(-0.01))} 0" rpy="0 0 0"/>
 			</visual>
-			<!--
-			   	<visual>
-		   			<geometry>
-						 <box size="0.06 0.06 0.06"/>
-		   			</geometry>
-					<origin xyz="${reflectx*(0.01)} ${ (reflecty*(-0.01))} -0.0128"/>
-		   		</visual>
-			-->
 		   	<collision>
 	   			<geometry>
@@ -125,12 +97,4 @@
 			    <origin xyz="0 0.0287 0" rpy="${reflectx*(pi)} 0 0"/>
 			</visual>
-			<!--
-			   	<visual>
-		   			<geometry>
-						 <box size="0.0525 0.085 0.0254"/>
-		   			</geometry>
-					<origin xyz="0 0.028 0"/>
-		   		</visual>
-			-->
 		   	<collision>
 	   			<geometry>
@@ -165,12 +129,4 @@
 		        <origin xyz="0.0 0 -0.067" rpy="-${pi/2} 0 ${reflectx*(-(pi/2))}"/>
 			</visual>
-			<!--
-			   	<visual>
-		   			<geometry>
-						 <box size="0.0525 0.0254 0.115"/>
-		   			</geometry>
-					<origin xyz="${reflectx*(0.02)} 0 -0.039"/>
-		   		</visual>
-			-->
 		   	<collision>
 	   			<geometry>
@@ -197,12 +153,4 @@
 				<origin xyz="0 0.0185 -0.0272" rpy="${pi/2} 0 ${pi}" />
 			</visual>
-			<!--
-			   	<visual>
-		   			<geometry>
-						 <box size="0.0523 0.0508 0.0400"/>
-		   			</geometry>
-					<origin xyz="0 0.01 -0.0072"/>
-		   		</visual>
-			-->
 		   	<collision>
 	   			<geometry>

Commit message: qp4-v2 model

File: src/qp4_description/urdf/qp4.urdf (robot description, URDF)
Before this commit: robot qp4, 18 links, 17 joints
Links:
- link back_left_femur_link: geometry collision box size=0.0508 0.0508 0.12065; visual mesh filename=file:///home/stewart/Robotics/ros-qp4/src/qp4_description/.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 scale=0.001 0.001 0.001
- link back_left_foot_link: geometry collision box size=0.0508 0.04445 0.0381; visual mesh filename=file:///home/stewart/Robotics/ros-qp4/src/qp4_description/.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 scale=0.001 0.001 0.001
- link back_left_hip_link: geometry collision box size=0.0381 0.0508 0.04445; visual mesh filename=file:///home/stewart/Robotics/ros-qp4/src/qp4_description/.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 scale=0.001 0.001 0.001
- link back_left_tibia_link: geometry collision box size=0.0508 0.0254 0.1143; visual mesh filename=file:///home/stewart/Robotics/ros-qp4/src/qp4_description/.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 scale=0.001 0.001 0.001
- link back_right_femur_link: geometry collision box size=0.0508 0.0508 0.12065; visual mesh filename=file:///home/stewart/Robotics/ros-qp4/src/qp4_description/.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 scale=0.001 0.001 0.001
- link back_right_foot_link: geometry collision box size=0.0508 0.04445 0.0381; visual mesh filename=file:///home/stewart/Robotics/ros-qp4/src/qp4_description/.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 scale=0.001 0.001 0.001
- link back_right_hip_link: geometry collision box size=0.0381 0.0508 0.04445; visual mesh filename=file:///home/stewart/Robotics/ros-qp4/src/qp4_description/.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 scale=0.001 0.001 0.001
- link back_right_tibia_link: geometry collision box size=0.0508 0.0254 0.1143; visual mesh filename=file:///home/stewart/Robotics/ros-qp4/src/qp4_description/.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 scale=0.001 0.001 0.001
- link front_left_femur_link: geometry collision box size=0.0508 0.0508 0.12065; visual mesh filename=file:///home/stewart/Robotics/ros-qp4/src/qp4_description/.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 scale=0.001 0.001 0.001
- link front_left_foot_link: geometry collision box size=0.0508 0.04445 0.0381; visual mesh filename=file:///home/stewart/Robotics/ros-qp4/src/qp4_description/.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 scale=0.001 0.001 0.001
- link front_left_hip_link: geometry collision box size=0.0381 0.0508 0.04445; visual mesh filename=file:///home/stewart/Robotics/ros-qp4/src/qp4_description/.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 scale=0.001 0.001 0.001
- link front_left_tibia_link: geometry collision box size=0.0508 0.0254 0.1143; visual mesh filename=file:///home/stewart/Robotics/ros-qp4/src/qp4_description/.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 scale=0.001 0.001 0.001
- link front_right_femur_link: geometry collision box size=0.0508 0.0508 0.12065; visual mesh filename=file:///home/stewart/Robotics/ros-qp4/src/qp4_description/.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 scale=0.001 0.001 0.001
- link front_right_foot_link: geometry collision box size=0.0508 0.04445 0.0381; visual mesh filename=file:///home/stewart/Robotics/ros-qp4/src/qp4_description/.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 scale=0.001 0.001 0.001
- link front_right_hip_link: geometry collision box size=0.0381 0.0508 0.04445; visual mesh filename=file:///home/stewart/Robotics/ros-qp4/src/qp4_description/.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 scale=0.001 0.001 0.001
- link front_right_tibia_link: geometry collision box size=0.0508 0.0254 0.1143; visual mesh filename=file:///home/stewart/Robotics/ros-qp4/src/qp4_description/.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 scale=0.001 0.001 0.001
- link torso_link: geometry collision box size=0.0762 0.3048 0.0254; collision box size=0.1016 0.0508 0.0254
Joints:
- joint back_left_ankle_joint: origin xyz=-0.0185 -0.0002 -0.077 rpy=0 0 0 -> xyz=0 0 -0.0762 rpy=0 0 0
- joint back_left_hip_lateral_joint: axis (none) -> 1 0 0; child back_left_femur_link -> back_left_hip_link; origin xyz=-0.0192 0.0005 -0.0290 rpy=-1.57079632679 0 0 -> xyz=-0.053975 -0.127 -0.0254 rpy=0 0 0; parent back_left_hip_link -> torso_link
- joint back_left_hip_swing_joint: child back_left_hip_link -> back_left_femur_link; origin xyz=-0.0395 -0.1095 -0.0315 rpy=0 0 0 -> xyz=-0.0254 0 0.01905 rpy=0 0 0; parent torso_link -> back_left_hip_link
- joint back_left_knee_joint: axis (none) -> 1 0 0; origin xyz=0.019 0.0572 0 rpy=1.57079632679 0 0 -> xyz=0 0 -0.0889 rpy=0 0 0
- joint back_right_ankle_joint: origin xyz=0.0185 -0.0002 -0.077 rpy=0 0 0 -> xyz=0 0 -0.0762 rpy=0 0 0
- joint back_right_hip_lateral_joint: axis (none) -> 1 0 0; child back_right_femur_link -> back_right_hip_link; origin xyz=0.0192 0.0005 -0.0290 rpy=-1.57079632679 0 0 -> xyz=0.053975 -0.127 -0.0254 rpy=0 0 0; parent back_right_hip_link -> torso_link
- joint back_right_hip_swing_joint: child back_right_hip_link -> back_right_femur_link; origin xyz=0.0395 -0.1095 -0.0315 rpy=0 0 0 -> xyz=0.0254 0 0.01905 rpy=0 0 0; parent torso_link -> back_right_hip_link
- joint back_right_knee_joint: axis (none) -> 1 0 0; origin xyz=-0.019 0.0572 0 rpy=1.57079632679 0 0 -> xyz=0 0 -0.0889 rpy=0 0 0
- joint front_left_ankle_joint: origin xyz=-0.0185 0.0002 -0.077 rpy=0 0 0 -> xyz=0 0 -0.0762 rpy=0 0 0
- joint front_left_hip_lateral_joint: axis (none) -> 1 0 0; child front_left_femur_link -> front_left_hip_link; origin xyz=-0.0192 0.0005 -0.0290 rpy=-1.57079632679 0 0 -> xyz=-0.053975 0.127 -0.0254 rpy=0 0 0; parent front_left_hip_link -> torso_link
- joint front_left_hip_swing_joint: child front_left_hip_link -> front_left_femur_link; origin xyz=-0.0395 0.1095 -0.0315 rpy=0 0 0 -> xyz=-0.0254 0 0.01905 rpy=0 0 0; parent torso_link -> front_left_hip_link
- joint front_left_knee_joint: axis (none) -> 1 0 0; origin xyz=0.019 0.0572 0 rpy=1.57079632679 0 0 -> xyz=0 0 -0.0889 rpy=0 0 0
- joint front_right_ankle_joint: origin xyz=0.0185 0.0002 -0.077 rpy=0 0 0 -> xyz=0 0 -0.0762 rpy=0 0 0
- joint front_right_hip_lateral_joint: axis (none) -> 1 0 0; child front_right_femur_link -> front_right_hip_link; origin xyz=0.0192 0.0005 -0.0290 rpy=-1.57079632679 0 0 -> xyz=0.053975 0.127 -0.0254 rpy=0 0 0; parent front_right_hip_link -> torso_link
- joint front_right_hip_swing_joint: child front_right_hip_link -> front_right_femur_link; origin xyz=0.0395 0.1095 -0.0315 rpy=0 0 0 -> xyz=0.0254 0 0.01905 rpy=0 0 0; parent torso_link -> front_right_hip_link
- joint front_right_knee_joint: axis (none) -> 1 0 0; origin xyz=-0.019 0.0572 0 rpy=1.57079632679 0 0 -> xyz=0 0 -0.0889 rpy=0 0 0

File: src/qp4_description/urdf/qp4.xacro (robot description, xacro)
@@ -12,7 +12,10 @@
         <axis xyz="0 0 1"/>
     </xacro:macro>
-    <xacro:include filename="$(find qp4_description)/urdf/qp4_materials.xacro"/>
+	<xacro:include filename="$(find qp4_description)/urdf/qp4_materials.xacro"/>
+<!--
     <xacro:include filename="$(find qp4_description)/urdf/qp4_gazebo.xacro"/>
     <xacro:include filename="$(find qp4_description)/urdf/qp4_parts.xacro"/>
+-->
+    <xacro:include filename="$(find qp4_description)/urdf/qp4_parts_v2.xacro"/>
 	<link name="base_link"></link>
  	<joint name="base_to_torso" type="fixed">
